Commit message: added dds qos config

File: ros2_driver/urdf/ur.urdf.xacro (robot description, xacro)
@@ -4,5 +4,5 @@
   <xacro:arg name="name" default="ur"/>
   <!-- ur_description -->
-  <xacro:include filename="$(find ur_description)/urdf/ur_macro.xacro"/>
+  <xacro:include filename="$(find octa_ros)/urdf/ur_macro.xacro"/>
   <!-- ros2 control include -->
   <xacro:include filename="$(find ur_robot_driver)/urdf/ur.ros2_control.xacro" />

File: ros2_driver/urdf/ur_end_effector.xacro (robot description, xacro)
@@ -98,5 +98,5 @@
   />
   <xacro:end_effector prefix="" parent="wrist_3_link">
-    <origin xyz="0 0.014 0.1328" rpy="0 0 0"/>
+    <origin xyz="0.00015 0.014 0.1328" rpy="0 0 0"/>
   </xacro:end_effector>
 </robot>

File: ros2_driver/urdf/ur_macro.xacro (robot description, xacro)
@@ -306,5 +306,6 @@
     <joint name="${tf_prefix}flange-tool0" type="fixed">
       <!-- default toolframe - X+ left, Y+ up, Z+ front -->
-      <origin xyz="0 0 0" rpy="${pi/2.0} 0 ${pi/2.0}"/>
+      <!-- origin xyz="0 0 0" rpy="${pi/2.0} 0 ${pi/2.0}"/ -->
+      <origin xyz="0.000015 0.014 0.1328" rpy="${pi/2.0} 0 ${pi/2.0}"/>
       <parent link="${tf_prefix}flange"/>
       <child link="${tf_prefix}tool0"/>

Commit message: tcp center correction and free drive mode addition

File: ros2_driver/urdf/ur.urdf.xacro (robot description, xacro)
@@ -98,5 +98,5 @@
   />
   <xacro:end_effector prefix="" parent="flange">
-    <origin xyz="0.0626 0.0 0.0" rpy="0 0 0"/>
+    <origin xyz="0.0501 0.0 0.0" rpy="0 0 0"/>
   </xacro:end_effector>
 </robot>

File: ros2_driver/urdf/ur_macro.xacro (robot description, xacro)
@@ -307,5 +307,6 @@
       <!-- default toolframe - X+ left, Y+ up, Z+ front -->
       <!-- origin xyz="0 0 0" rpy="${pi/2.0} 0 ${pi/2.0}"/ -->
-      <origin xyz="0.132806 0.008578264656 0.008578264656" rpy="${pi/2.0} ${pi/4.0} ${pi/2.0}"/>
+      <!-- <origin xyz="0.132806 0.008578264656 0.008578264656" rpy="${pi/2.0} ${pi/4.0} ${pi/2.0}"/> -->
+      <origin xyz="0.132806 0.0089552395 0.0089552395" rpy="${pi/2.0} ${pi/4.0} ${pi/2.0}"/>
       <parent link="${tf_prefix}flange"/>
       <child link="${tf_prefix}tool0"/>

Commit message: semi-stable version

File: ros2_driver/urdf/ur.urdf.xacro (robot description, xacro)
@@ -98,5 +98,5 @@
   />
   <xacro:end_effector prefix="" parent="flange">
-    <origin xyz="0.0501 0.0 0.0" rpy="0 0 0"/>
+    <origin xyz="0.051 0.0 0.0" rpy="0 0 0"/>
   </xacro:end_effector>
 </robot>

File: ros2_driver/urdf/ur_macro.xacro (robot description, xacro)
@@ -308,5 +308,5 @@
       <!-- origin xyz="0 0 0" rpy="${pi/2.0} 0 ${pi/2.0}"/ -->
       <!-- <origin xyz="0.132806 0.008578264656 0.008578264656" rpy="${pi/2.0} ${pi/4.0} ${pi/2.0}"/> -->
-      <origin xyz="0.132806 0.0089552395 0.0089552395" rpy="${pi/2.0} ${pi/4.0} ${pi/2.0}"/>
+      <origin xyz="0.132806 0.008578264656 0.008578264656" rpy="${pi/2.0} ${pi/4.0} ${pi/2.0}"/>
       <parent link="${tf_prefix}flange"/>
       <child link="${tf_prefix}tool0"/>
