Commit message: fixed tcp

File: ros2_driver/urdf/ur_macro.xacro (robot description, xacro)
@@ -307,5 +307,6 @@
       <!-- default toolframe - X+ left, Y+ up, Z+ front -->
       <!-- origin xyz="0 0 0" rpy="${pi/2.0} 0 ${pi/2.0}"/ -->
-      <origin xyz="0.000015 0.014 0.1328" rpy="${pi/2.0} 0 ${pi/2.0}"/>
+      <!-- origin xyz="0.000015 0.014 0.1328" rpy="${pi/2.0} 0 ${pi/2.0}"/ -->
+      <origin xyz="0.1328 -0.000015 -0.014" rpy="${pi/2.0} 0 ${pi/2.0}"/>
       <parent link="${tf_prefix}flange"/>
       <child link="${tf_prefix}tool0"/>

Commit message: fine-tuned tcp

File: ros2_driver/urdf/ur_macro.xacro (robot description, xacro)
@@ -308,5 +308,5 @@
       <!-- origin xyz="0 0 0" rpy="${pi/2.0} 0 ${pi/2.0}"/ -->
       <!-- origin xyz="0.000015 0.014 0.1328" rpy="${pi/2.0} 0 ${pi/2.0}"/ -->
-      <origin xyz="0.1328 -0.000015 -0.014" rpy="${pi/2.0} 0 ${pi/2.0}"/>
+      <origin xyz="0.1328 -0.001985 0.011968" rpy="${pi/2.0} 0 ${pi/2.0}"/>
       <parent link="${tf_prefix}flange"/>
       <child link="${tf_prefix}tool0"/>

Commit message: bug fixes, refinement, and TCP adjustment

File: ros2_driver/urdf/ur_macro.xacro (robot description, xacro)
@@ -307,5 +307,5 @@
       <!-- default toolframe - X+ left, Y+ up, Z+ front -->
       <!-- origin xyz="0 0 0" rpy="${pi/2.0} 0 ${pi/2.0}"/ -->
-      <origin xyz="0.132806 -0.008578264656 0.008578264656" rpy="${pi/2.0} ${pi/4.0} ${pi/2.0}"/>
+      <origin xyz="0.132806 0.008578264656 0.008578264656" rpy="${pi/2.0} ${pi/4.0} ${pi/2.0}"/>
       <parent link="${tf_prefix}flange"/>
       <child link="${tf_prefix}tool0"/>

Commit message: current tcp correction, added docker files, and cleanup

File: ros2_driver/urdf/ur_macro.xacro (robot description, xacro)
@@ -308,5 +308,5 @@
       <!-- origin xyz="0 0 0" rpy="${pi/2.0} 0 ${pi/2.0}"/ -->
       <!-- <origin xyz="0.132806 0.008578264656 0.008578264656" rpy="${pi/2.0} ${pi/4.0} ${pi/2.0}"/> -->
-      <origin xyz="0.132806 0.008578264656 0.008578264656" rpy="${pi/2.0} ${pi/4.0} ${pi/2.0}"/>
+      <origin xyz="0.132806 0.008866893596 0.007878663464" rpy="${pi/2.0} ${pi/4.0} ${pi/2.0}"/>
       <parent link="${tf_prefix}flange"/>
       <child link="${tf_prefix}tool0"/>

Commit message: working tcp, freedrive bug fix, autofocus slow-fast axis bug

File: ros2_driver/urdf/ur_macro.xacro (robot description, xacro)
@@ -308,5 +308,5 @@
       <!-- origin xyz="0 0 0" rpy="${pi/2.0} 0 ${pi/2.0}"/ -->
       <!-- <origin xyz="0.132806 0.008578264656 0.008578264656" rpy="${pi/2.0} ${pi/4.0} ${pi/2.0}"/> -->
-      <origin xyz="0.132806 0.008866893596 0.007878663464" rpy="${pi/2.0} ${pi/4.0} ${pi/2.0}"/>
+      <origin xyz="0.132806 0.008412086 0.007853472611" rpy="${pi/2.0} ${pi/4.0} ${pi/2.0}"/>
       <parent link="${tf_prefix}flange"/>
       <child link="${tf_prefix}tool0"/>

Commit message: formatting

File: ros2_driver/urdf/ur_macro.xacro (robot description, xacro)
@@ -307,5 +307,4 @@
       <!-- default toolframe - X+ left, Y+ up, Z+ front -->
       <!-- origin xyz="0 0 0" rpy="${pi/2.0} 0 ${pi/2.0}"/ -->
-      <!-- <origin xyz="0.132806 0.008578264656 0.008578264656" rpy="${pi/2.0} ${pi/4.0} ${pi/2.0}"/> -->
       <origin xyz="0.132806 0.008412086 0.007853472611" rpy="${pi/2.0} ${pi/4.0} ${pi/2.0}"/>
       <parent link="${tf_prefix}flange"/>

Commit message: bugfixes on axis delay

File: ros2_driver/urdf/ur_macro.xacro (robot description, xacro)
@@ -307,5 +307,6 @@
       <!-- default toolframe - X+ left, Y+ up, Z+ front -->
       <!-- origin xyz="0 0 0" rpy="${pi/2.0} 0 ${pi/2.0}"/ -->
-      <origin xyz="0.132806 0.008412086 0.007853472611" rpy="${pi/2.0} ${pi/4.0} ${pi/2.0}"/>
+      <!--origin xyz="0.132806 0.008412086 0.007853472611" rpy="${pi/2.0} ${pi/4.0} ${pi/2.0}"/ -->
+      <origin xyz="0.132806 0.008687832114 0.008129217757" rpy="${pi/2.0} ${pi/4.0} ${pi/2.0}"/>
       <parent link="${tf_prefix}flange"/>
       <child link="${tf_prefix}tool0"/>
