Commit message: added tcp

File: ros2_driver/urdf/end_effector.xacro (robot description, xacro)
@@ -12,5 +12,5 @@
       <visual>
         <geometry>
-          <sphere radius="0.05"/>
+          <sphere radius="0.01"/>
         </geometry>
         <material name="blue">

File: ros2_driver/urdf/ur_end_effector.xacro (robot description, xacro)
@@ -98,5 +98,5 @@
   />
   <xacro:end_effector prefix="" parent="wrist_3_link">
-    <origin xyz="0 0 0.04" rpy="0 0 0"/>
+    <origin xyz="0 0.014 0.1328" rpy="0 0 0"/>
   </xacro:end_effector>
 </robot>

Commit message: bugfixes for tcp and added stl files for end_effector

File: ros2_driver/urdf/end_effector.xacro (robot description, xacro)
@@ -12,5 +12,5 @@
       <visual>
         <geometry>
-          <sphere radius="0.01"/>
+          <sphere radius="0.0625"/>
         </geometry>
         <material name="blue">
@@ -20,5 +20,5 @@
       <collision>
         <geometry>
-          <sphere radius="0.03"/>
+          <sphere radius="0.0625"/>
         </geometry>
       </collision>

File: ros2_driver/urdf/ur.urdf.xacro (robot description, xacro)
@@ -8,4 +8,6 @@
   <xacro:include filename="$(find ur_robot_driver)/urdf/ur.ros2_control.xacro" />
   <xacro:include filename="$(find ur_description)/urdf/inc/ur_transmissions.xacro" />
+  <!-- end_effector include -->
+  <xacro:include filename="$(find octa_ros)/urdf/end_effector.xacro" />
   <!-- possible 'ur_type' values: ur3, ur3e, ur5, ur5e, ur10, ur10e, ur16e, ur20 -->
   <!-- the default value should raise an error in case this was called without defining the type -->
@@ -95,3 +97,6 @@
     trajectory_port="$(arg trajectory_port)"
   />
+  <xacro:end_effector prefix="" parent="flange">
+    <origin xyz="0.0626 0.0 0.0" rpy="0 0 0"/>
+  </xacro:end_effector>
 </robot>

File: ros2_driver/urdf/ur_macro.xacro (robot description, xacro)
@@ -307,6 +307,5 @@
       <!-- default toolframe - X+ left, Y+ up, Z+ front -->
       <!-- origin xyz="0 0 0" rpy="${pi/2.0} 0 ${pi/2.0}"/ -->
-      <!-- origin xyz="0.000015 0.014 0.1328" rpy="${pi/2.0} 0 ${pi/2.0}"/ -->
-      <origin xyz="0.1328 -0.001985 0.011968" rpy="${pi/2.0} 0 ${pi/2.0}"/>
+      <origin xyz="0.132806 -0.008578264656 0.008578264656" rpy="${pi/2.0} ${pi/4.0} ${pi/2.0}"/>
       <parent link="${tf_prefix}flange"/>
       <child link="${tf_prefix}tool0"/>

Commit message: z-axis working version

File: ros2_driver/urdf/end_effector.xacro (robot description, xacro)
@@ -12,7 +12,7 @@
       <visual>
         <geometry>
-          <sphere radius="0.0625"/>
+          <sphere radius="0.05"/>
         </geometry>
-        <material name="blue">
+	<material name="green">
           <color rgba="0 0 1 1"/>
         </material>
@@ -20,5 +20,5 @@
       <collision>
         <geometry>
-          <sphere radius="0.0625"/>
+          <sphere radius="0.05"/>
         </geometry>
       </collision>

Commit message: tcp and slow axis fix

File: ros2_driver/urdf/end_effector.xacro (robot description, xacro)
@@ -12,5 +12,5 @@
       <visual>
         <geometry>
-          <sphere radius="0.05"/>
+          <sphere radius="0.06"/>
         </geometry>
 	<material name="green">

File: ros2_driver/urdf/oct_setup.xacro (robot description, xacro)
@@ -102,5 +102,5 @@
     <!-- origin xyz="0 0 0" rpy="${pi/2.0} 0 ${pi/2.0}"/ -->
     <!-- <origin xyz="0.132806 0.008687832114 0.008129217757" rpy="${pi/2.0} ${pi/4.0} ${pi/2.0}"/> -->
-    <origin xyz="0.008687832114 0.008129217757 0.132806" rpy="0 0 ${-3*pi/4.0}"/>
+    <origin xyz="0.010687832114 0.010129217757 0.132806" rpy="0 0 ${-3*pi/4.0}"/>
     <parent link="$(arg tf_prefix)tool0"/>
     <child link="$(arg tf_prefix)tcp"/>
