Commit message: reinitialized tcp and adjusted docker files

File: urdf/oct_setup.xacro (robot description, xacro)
@@ -110,10 +110,10 @@
   </link>
   <joint name="$(arg tf_prefix)tool0-oct" type="fixed">
-    <origin xyz="0.0104474865 0.00835817192 0.132806" rpy="0 0 ${-3*pi/4.0}"/>
+    <origin xyz="0.00 0.00 0.132806" rpy="0 0 ${-3*pi/4.0}"/>
     <parent link="$(arg tf_prefix)tool0"/>
     <child link="$(arg tf_prefix)oct"/>
   </joint>
   <joint name="$(arg tf_prefix)oct-tcp" type="fixed">
-    <origin xyz="0.00047 -0.00013 0.0" rpy="0 0 0"/>
+    <origin xyz="0.000 0.000 0.0" rpy="0 0 0"/>
     <parent link="$(arg tf_prefix)oct"/>
     <child link="$(arg tf_prefix)tcp"/>

Commit message: added back tcp and cleanup

File: urdf/oct_setup.xacro (robot description, xacro)
@@ -110,10 +110,10 @@
   </link>
   <joint name="$(arg tf_prefix)tool0-oct" type="fixed">
-    <origin xyz="0.00 0.00 0.132806" rpy="0 0 ${-3*pi/4.0}"/>
+    <origin xyz="0.0104474865 0.00835817192 0.132806" rpy="0 0 ${-3*pi/4.0}"/>
     <parent link="$(arg tf_prefix)tool0"/>
     <child link="$(arg tf_prefix)oct"/>
   </joint>
   <joint name="$(arg tf_prefix)oct-tcp" type="fixed">
-    <origin xyz="0.000 0.000 0.0" rpy="0 0 0"/>
+    <origin xyz="0.00137 -0.0013 0.0" rpy="0 0 0"/>
     <parent link="$(arg tf_prefix)oct"/>
     <child link="$(arg tf_prefix)tcp"/>

Commit message: cleanup and realign tcp

File: urdf/oct_setup.xacro (robot description, xacro)
@@ -115,5 +115,5 @@
   </joint>
   <joint name="$(arg tf_prefix)oct-tcp" type="fixed">
-    <origin xyz="0.00137 -0.0013 0.0" rpy="0 0 0"/>
+    <origin xyz="0.00137 0.00104 0.0" rpy="0 0 0"/>
     <parent link="$(arg tf_prefix)oct"/>
     <child link="$(arg tf_prefix)tcp"/>

Commit message: changed z angle planner and reinitialized tcp

File: urdf/oct_setup.xacro (robot description, xacro)
@@ -115,5 +115,5 @@
   </joint>
   <joint name="$(arg tf_prefix)oct-tcp" type="fixed">
-    <origin xyz="0.00137 0.00104 0.0" rpy="0 0 0"/>
+    <origin xyz="0.00047 -0.00013 0.0" rpy="0 0 0"/>
     <parent link="$(arg tf_prefix)oct"/>
     <child link="$(arg tf_prefix)tcp"/>

Commit message: recalibrate tcp and bug fixes

File: urdf/oct_setup.xacro (robot description, xacro)
@@ -115,5 +115,5 @@
   </joint>
   <joint name="$(arg tf_prefix)oct-tcp" type="fixed">
-    <origin xyz="0.00047 -0.00013 0.0" rpy="0 0 0"/>
+    <origin xyz="-0.00008 -0.00023 0.0" rpy="0 0 0"/>
     <parent link="$(arg tf_prefix)oct"/>
     <child link="$(arg tf_prefix)tcp"/>

Commit message: hard code pipelines and calibrate tcp

File: urdf/oct_setup.xacro (robot description, xacro)
@@ -115,5 +115,5 @@
   </joint>
   <joint name="$(arg tf_prefix)oct-tcp" type="fixed">
-    <origin xyz="-0.00008 -0.00023 0.0" rpy="0 0 0"/>
+    <origin xyz="0.0005989 -0.0011181 0.0" rpy="0 0 0"/>
     <parent link="$(arg tf_prefix)oct"/>
     <child link="$(arg tf_prefix)tcp"/>
