Commit message: new xacro structure

File: urdf/end_effector.xacro (robot description, xacro)
@@ -2,5 +2,4 @@
 <robot xmlns:xacro="http://www.ros.org/wiki/xacro">
   <xacro:macro name="end_effector" params="prefix parent *origin">
-    <!-- Joint connecting to parent link -->
     <joint name="${prefix}end_effector_joint" type="fixed">
       <parent link="${parent}"/>
@@ -8,22 +7,27 @@
       <xacro:insert_block name="origin"/>
     </joint>
-    <!-- End effector link -->
     <link name="${prefix}end_effector_link">
       <visual>
+        <origin xyz="0 0 0" rpy="0 0 0" />
         <geometry>
-          <sphere radius="0.06"/>
+          <mesh filename="package://octa_ros/urdf/end_effector.stl" />
         </geometry>
-	<material name="green">
-          <color rgba="0 0 1 1"/>
+        <material name="oct_end_effector">
+          <color rgba="0.0 0.3 0.8 1.0"/>
         </material>
       </visual>
       <collision>
+        <origin xyz="0 0 0" rpy="0 0 0" />
         <geometry>
-          <sphere radius="0.05"/>
+          <mesh filename="package://octa_ros/urdf/end_effector.stl" />
         </geometry>
       </collision>
       <inertial>
-        <mass value="0.1"/>
-        <inertia ixx="0.000016667" ixy="0" ixz="0" iyy="0.000016667" iyz="0" izz="0.000016667"/>
+        <origin xyz="0.00632 -0.04819 0.08954" rpy="0 0 0" />
+        <mass value="0.4376"/>
+        <inertia
+          ixx="0.000563" ixy="0.0000074" ixz="0.000074"
+          iyy="0.000636" iyz="-0.000059"
+          izz="0.000322"/>
       </inertial>
     </link>

File: urdf/oct_setup.xacro (robot description, xacro)
@@ -1,17 +1,17 @@
 <?xml version="1.0"?>
 <robot xmlns:xacro="http://wiki.ros.org/xacro" name="$(arg name)">
-  <!-- robot name parameter -->
-  <xacro:arg name="name" default="ur"/>
+  <!--
+    Built on top of ur_robot_driver/urdf/ur.urdf.xacro and only adds the OCT/TCP
+    assembly provided by octa_ros_tooling.
+  -->
+  <!-- Upstream UR definitions -->
   <xacro:include filename="$(find ur_description)/urdf/ur_macro.xacro"/>
-  <!-- ros2 control include -->
   <xacro:include filename="$(find ur_robot_driver)/urdf/ur.ros2_control.xacro" />
   <xacro:include filename="$(find ur_description)/urdf/inc/ur_transmissions.xacro" />
-  <!-- end_effector include -->
-  <xacro:include filename="$(find octa_ros)/urdf/end_effector.xacro" />
-  <!-- <xacro:include filename="$(find ur_robot_driver)/urdf/ur.urdf.xacro" /> -->
-  <!-- possible 'ur_type' values: ur3, ur3e, ur5, ur5e, ur10, ur10e, ur16e, ur20 -->
-  <!-- the default value should raise an error in case this was called without defining the type -->
+  <!-- OCT-specific attachments -->
+  <xacro:include filename="$(find octa_ros)/urdf/oct_tooling.xacro" />
+  <!-- Pass-through UR driver arguments -->
+  <xacro:arg name="name" default="ur"/>
   <xacro:arg name="ur_type" default="urXe"/>
-  <!-- parameters -->
   <xacro:arg name="tf_prefix" default="" />
   <xacro:arg name="joint_limit_params" default="$(find ur_description)/config/$(arg ur_type)/joint_limits.yaml"/>
@@ -23,5 +23,4 @@
   <xacro:arg name="safety_pos_margin" default="0.15"/>
   <xacro:arg name="safety_k_position" default="20"/>
-  <!-- ros2_control related parameters -->
   <xacro:arg name="headless_mode" default="false" />
   <xacro:arg name="robot_ip" default="0.0.0.0" />
@@ -34,5 +33,4 @@
   <xacro:arg name="script_sender_port" default="50002"/>
   <xacro:arg name="trajectory_port" default="50003"/>
-  <!--   tool communication related parameters-->
   <xacro:arg name="use_tool_communication" default="false" />
   <xacro:arg name="tool_voltage" default="0" />
@@ -44,13 +42,10 @@
   <xacro:arg name="tool_device_name" default="/tmp/ttyUR" />
   <xacro:arg name="tool_tcp_port" default="54321" />
-  <!-- Simulation parameters -->
   <xacro:arg name="use_mock_hardware" default="false" />
   <xacro:arg name="mock_sensor_commands" default="false" />
   <xacro:arg name="simulation_controllers" default="" />
-  <!-- initial position for simulations (Mock Hardware, Gazebo, Ignition) -->
   <xacro:arg name="initial_positions_file" default="$(find ur_description)/config/initial_positions.yaml"/>
-  <!-- convert to property to use substitution in function -->
+  <!-- Derived properties reused below -->
   <xacro:property name="initial_positions_file" default="$(arg initial_positions_file)"/>
-  <!-- create link fixed to the "world" -->
   <link name="world" />
   <xacro:ur_robot
@@ -64,9 +59,7 @@
       safety_limits="$(arg safety_limits)"
       safety_pos_margin="$(arg safety_pos_margin)"
-      safety_k_position="$(arg safety_k_position)"
-      >
-    <origin xyz="0 0 0" rpy="0 0 0" />          <!-- position robot in the world -->
+      safety_k_position="$(arg safety_k_position)">
+    <origin xyz="0 0 0" rpy="0 0 0" />
   </xacro:ur_robot>
-  <!-- ros2 control instance -->
   <xacro:ur_ros2_control
       name="$(arg name)"
@@ -95,30 +88,5 @@
       reverse_port="$(arg reverse_port)"
       script_sender_port="$(arg script_sender_port)"
-      trajectory_port="$(arg trajectory_port)"
-      />
-  <link name="$(arg tf_prefix)oct"/>
-  <link name="$(arg tf_prefix)tcp">
-    <inertial>
-      <origin xyz="0 0 0.051" rpy="0 0 0" />
-      <mass value="2.0" />
-      <inertia
-          ixx="0.0005" ixy="0" ixz="0"
-          iyy="0.0005" iyz="0"
-          izz="0.0005"
-          />
-    </inertial>
-  </link>
-  <joint name="$(arg tf_prefix)tool0-oct" type="fixed">
-    <origin xyz="0.0104474865 0.00835817192 0.132806" rpy="0 0 ${-3*pi/4.0}"/>
-    <parent link="$(arg tf_prefix)tool0"/>
-    <child link="$(arg tf_prefix)oct"/>
-  </joint>
-  <joint name="$(arg tf_prefix)oct-tcp" type="fixed">
-    <origin xyz="0.0005989 -0.0011181 0.0" rpy="0 0 0"/>
-    <parent link="$(arg tf_prefix)oct"/>
-    <child link="$(arg tf_prefix)tcp"/>
-  </joint>
-  <xacro:end_effector prefix="" parent="$(arg tf_prefix)tcp">
-    <origin xyz="0.0 0.0 -0.08" rpy="0 0 0"/>
-  </xacro:end_effector>
+      trajectory_port="$(arg trajectory_port)"/>
+  <xacro:octa_ros_tooling tf_prefix="$(arg tf_prefix)" />
 </robot>
